Commit message: Switched to the latest urdf model
- Latest urdf model considered
- Latest meshes considered

File: src/adherent/model/iCubGazeboV3_xsens/iCubGazeboV3_xsens.urdf (robot description, URDF)
Before this commit: robot iCub3, 60 links, 59 joints
Links:
- added link imu_frame
Joints:
- added joint imu_frame_fixed_joint: type fixed, parent head, child imu_frame, origin xyz=0.0034999999997785457 0.0054999999863750895 0.1013340000004441 rpy=-3.141592653589793 0 -1.570796326794897
- joint r_wrist_yaw: limit (none) -> lower=-0.2617993877991494 upper=0.6108652381980153 effort=50000 velocity=120.0; type continuous -> revolute
